File: models/PCB/Untitled.kicad_sch (KiCad schematic)
At the start: 24 parts, among them J2 Screw_Terminal_01x02, J3 Conn_01x03_Pin, M1 Motor_DC, M2 Motor_Servo, Q1 BC547, SW1 SW_Push, SW2 SW_SPST, U1 VL53l1x, U2 VL53l1x, U3 VL53l1x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

Commit message: Team photos added
Parts:
- renumbered IC6 to RaspberryPi, U1 to VL53l1X
Other:
- note added: "Multiplexer"
- note added: "VL53l1x"
- note added: "XY-3606"
Changed lines of the file:
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@@
 	(generator_version "9.0")
 	(paper "A4")
+	(text "VL53l1x"
+		(exclude_from_sim no)
+		(at 71.628 16.764 0)
+		(effects
+			(font
+				(size 1.27 1.27)
+			)
+		)
+	)
+	(text "XY-3606\n"
+		(exclude_from_sim no)
+		(at 86.36 141.224 0)
+		(effects
+			(font
+				(size 1.27 1.27)
+			)
+		)
+	)
+	(text "Multiplexer\n"
+		(exclude_from_sim no)
+		(at 74.93 109.728 0)
+		(effects
+			(font
+				(size 1.27 1.27)
+			)
+		)
+	)
 	(junction
 		(at 119.38 130.81)
@@
 				)
 				(justify left)
+				(hide yes)
 			)
 		)
@@
 				)
 				(justify left)
+				(hide yes)
 			)
 		)
@@
 				)
 				(justify left)
+				(hide yes)
 			)
 		)
@@
 				)
 				(justify left)
+				(hide yes)
 			)
 		)
@@
 		(on_board yes)
 		(dnp no)
-		(fields_autoplaced yes)
-		(property "Reference" "IC6"
-			(at 161.29 76.2 0)
+		(property "Reference" "RaspberryPi"
+			(at 160.528 96.266 0)
 			(effects
 				(font
@@
 		)
 		(property "Value" "~"
-			(at 161.29 78.74 0)
+			(at 161.29 80.01 0)
 			(effects
 				(font
@@
 			(project ""
 				(path "/93becf76-4cbc-4b5f-b49a-c47e1799cb2f"
-					(reference "IC6")
+					(reference "RaspberryPi")
 					(unit 1)
 				)
@@
 		(dnp no)
 		(fields_autoplaced yes)
-		(property "Reference" "U1"
+		(property "Reference" "VL53l1X"
 			(at 69.85 20.32 0)
 			(effects
@@
 			(project ""
 				(path "/93becf76-4cbc-4b5f-b49a-c47e1799cb2f"
-					(reference "U1")
+					(reference "VL53l1X")
 					(unit 1)
 				)
@@
 					(size 1.27 1.27)
 				)
+				(hide yes)
 			)
 		)
